File: RelojAzul.sch (EAGLE design)
At the start: 6 parts, among them X1 5V cc.

Commit message: ESQUEMA
ESQUEMA 2
Parts:
- removed JP1, JP2, JP3: (no value), pinhead:PINHD-1X4
- removed SG1: F/CM04P, buzzer:F/CM04P
- added JP4, JP5, JP6: (no value), pinhead:PINHD-1X4
- added R1: 10K, resistor:R-EU_0204_5
- added R2: 4K7, resistor:R-EU_0204_5
- added S1: (no value), switch-omron:40-XX
- added SG2: F/CM04P, buzzer:F/CM04P
- added X2: DS1820, con-molex:22-23-2031
Connections:
- new net N$10: JP6.1, U$1.A6
- new net N$11: R2.1, U$1.*10, X2-2.S
- new net N$2: R1.1, S1.S, S1.S1, U$1.*6
- new net N$3: SG2.2, U$1.7
- new net N$4: JP4.4, U$1.2
- new net N$5: JP4.3, U$1.*3
- new net N$6: JP5.1, U$1.8
- new net N$7: JP5.2, U$1.*9
- new net N$9: JP6.2, U$1.A5
- net +5V: now also JP4.1, JP5.3, JP6.3, R1.2, R2.2, SG2.1, X2-1.S
- net GND: now also JP4.2, JP5.4, JP6.4, S1.P, U$1.GND, X2-3.S; no longer U$1.RST
Other:
- note added: "1"
- note added: "DATO"
- note added: "Display TM1637"
- note added: "Modulo Bluetooth HC-05"
- note added: "Modulo RTC DS3231"
- note added: "SCL"
- note added: "SDA"
- note added: "ck"
- note added: "dato"
- note added: "rx"
- note added: "tx"
- moved on the sheet: U$1, X1-1, X1-2
